File: RoboBlock/nano_bt.sch (EAGLE design)
At the start: 16 parts, among them IC1 L293D, M1 ARDUINO-NANO-3.0

Commit message: sensor
Parts:
- added S1: SPST, adafruit_arduino:SPST
Connections:
- new net N$12: DCV.1, S1.P
- net N$8: now also S1.S; no longer DCV.1
