File: RoboBlock/uno_bt.sch (EAGLE design)
At the start: 17 parts, among them IC1 L293D, U1 ARDUINOR3-DIMENSION

Commit message: sensor
Parts:
- U1: value ARDUINOR3-DIMENSION -> ARDUINOR3-BPLACE; device adafruit_arduino:ARDUINOR3-DIMENSION -> adafruit_arduino:ARDUINOR3-BPLACE
Changed lines of the file:
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@@
 <part name="HCSR04" library="pinhead" library_urn="urn:adsk.eagle:library:325" deviceset="PINHD-1X4" device="" package3d_urn="urn:adsk.eagle:package:22407/2"/>
 <part name="SG2" library="buzzer" library_urn="urn:adsk.eagle:library:113" deviceset="F/TMB" device="" package3d_urn="urn:adsk.eagle:package:5260/1"/>
-<part name="U1" library="adafruit_arduino" deviceset="ARDUINOR3" device="-DIMENSION"/>
+<part name="U1" library="adafruit_arduino" deviceset="ARDUINOR3" device="-BPLACE" value="ARDUINOR3-BPLACE"/>
 <part name="S1" library="adafruit_arduino" deviceset="SPST" device=""/>
 </parts>
