File: RoboBlock/sensor_potensio.sch (EAGLE design)
At the start: 2 parts

Commit message: printout pcb
Parts:
- added JP2, JP3, JP4, JP5, JP6: (no value), adafruit_arduino:PINHD-1X3
- added LDR: (no value), resistor:R-US_0204/5
- added LED1, LED2, LED3: (no value), adafruit_arduino:LED5MM
- added R1: 10K, adafruit_arduino:R-US_0207/7
- added R2, R3, R4: 220, adafruit_arduino:R-US_0207/7
- added SW1: (no value), adafruit_arduino:SWITCH_PUSHBUTTONEVQ-PE
- added TM2: (no value), adafruit_arduino:TRIM
Connections:
- new net N$1: JP2.3, R1.2, SW1.P$1
- new net N$10: LED2.A, R3.2
- new net N$11: JP5.2, R3.1
- new net N$12: LED3.A, R4.2
- new net N$13: JP5.3, LED2.C
- new net N$14: JP6.3, R4.1
- new net N$15: JP6.1, LED3.C
- new net N$2: JP2.1, R1.1
- new net N$3: JP2.2, SW1.P$2
- new net N$4: JP3.3, LDR.2, TM2.A
- new net N$5: JP3.1, TM2.E, TM2.S
- new net N$6: JP3.2, LDR.1
- new net N$7: LED1.A, R2.2
- new net N$8: JP4.3, R2.1
- new net N$9: JP4.1, LED1.C
Other:
- moved on the sheet: JP1, TM1
