File: RoboBlock/uno_bt.brd (EAGLE design)
At the start: 100 x 80 mm, 17 parts, among them IC1 L293D, U1 ARDUINOR3-DIMENSION

Commit message: sensor
Parts:
- U1: value ARDUINOR3-DIMENSION -> ARDUINOR3-BPLACE; device adafruit_arduino:ARDUINOR3 -> adafruit_arduino:ARDUINOR3-BPLACE
- moved IC1 18.0 mm to (25.4, 57.1)
Routing:
- net VIN: track 0.00 -> 69.1 mm
- net VCC: track 88.6 -> 108.7 mm
- net GND: track 104.0 -> 121.6 mm

Commit message: printout pcb
Parts:
- moved DCIN 63.3 mm to (20.3, 39.4)
- moved S1 61.6 mm to (31.8, 26.7)
- moved IC1 24.4 mm to (3.81, 68.6)
- moved BT1 12.8 mm to (80.0, 43.2)
- moved SG2 12.8 mm to (26.7, 55.9), turned to 90 degrees
- moved HCSR04 9.25 mm to (39.4, 50.8), turned to 270 degrees
- moved AN3 3.59 mm to (66.0, 30.5)
- moved AN4 3.59 mm to (74.9, 30.5)
- moved AN1 2.84 mm to (48.3, 30.5)
- moved AN2 2.84 mm to (57.1, 30.5)
- moved O1 2.84 mm to (48.3, 55.9), flipped to the top
- moved O2 2.84 mm to (57.1, 55.9)
- moved O3 2.84 mm to (66.0, 55.9)
- moved O4 2.84 mm to (74.9, 55.9)
Routing:
- net VIN: track 69.1 -> 0.00 mm
- net GND: track 121.6 -> 68.4 mm
- net VCC: track 108.7 -> 67.3 mm
- net D13: track 13.4 -> 0.00 mm
- net N$5: track 9.46 -> 0.00 mm
- net D0: track 32.6 -> 23.4 mm
- net D1: track 26.8 -> 19.1 mm
- net A0: track 23.5 -> 28.8 mm
- net A3: track 7.62 -> 12.0 mm
- net A2: track 12.5 -> 16.8 mm
- net A1: track 18.6 -> 22.4 mm
- net D10: track 9.84 -> 13.1 mm
- net D6: track 5.08 -> 8.15 mm
- net D9: track 5.19 -> 8.04 mm
- net D5: track 9.94 -> 12.0 mm
